Commit message: tested walking model

File: urdf/leg.urdf.xacro (robot description, xacro)
@@ -73,5 +73,5 @@
         </link>
         <gazebo reference="${leg}_hip_link">
-            <material>Gazebo/FlatBlack</material>
+            <material>Gazebo/White</material>
         </gazebo>
         <link name="${leg}_upper_leg_link">
@@ -139,5 +139,5 @@
         <joint name="${leg}_hip_joint" type="revolute">
             <axis xyz="1 0 0" />
-            <limit effort="25" lower="-${pi}" upper="${pi}" velocity="1.5" />
+            <limit effort="25" lower="-${pi}" upper="${pi}" velocity="3.0" />
             <parent link="base_link" />
             <child link="${leg}_hip_link" />
@@ -146,5 +146,5 @@
         <joint name="${leg}_upper_leg_joint" type="revolute">
             <axis xyz="0 1 0" />
-            <limit effort="25" lower="-${pi}" upper="${pi}" velocity="1.5" />
+            <limit effort="25" lower="-${pi}" upper="${pi}" velocity="3.0" />
             <parent link="${leg}_hip_link" />
             <child link="${leg}_upper_leg_link" />
@@ -153,5 +153,5 @@
         <joint name="${leg}_lower_leg_joint" type="revolute">
             <axis xyz="0 1 0" />
-            <limit effort="25" lower="-${pi}" upper="${pi}" velocity="1.5" />
+            <limit effort="25" lower="-${pi}" upper="${pi}" velocity="3.0" />
             <parent link="${leg}_upper_leg_link" />
             <child link="${leg}_lower_leg_link" />

File: urdf/opendog.urdf (robot description, URDF)
Before this commit: robot opendog, 29 links, 28 joints
Joints:
- joint base_link_to_base_inertia: origin xyz=0 0 0 rpy=0 0 0 -> xyz=0.05 0 0 rpy=0 0 0
- joint camera_joint: origin xyz=0.25 0.0 0.075 rpy=0 0 0 -> xyz=0.4 0.0 0.12 rpy=0 0 0
- joint hokuyo_joint: origin xyz=0.0 0.0 0.105 rpy=0 0 0 -> xyz=0.0 0.0 0.15 rpy=0 0 0
- joint lf_hip_joint: limit lower=-3.14159265359 upper=3.14159265359 effort=25 velocity=1.5 -> lower=-3.14159265359 upper=3.14159265359 effort=25 velocity=3.0
- joint lf_lower_leg_joint: limit lower=-3.14159265359 upper=3.14159265359 effort=25 velocity=1.5 -> lower=-3.14159265359 upper=3.14159265359 effort=25 velocity=3.0
- joint lf_upper_leg_joint: limit lower=-3.14159265359 upper=3.14159265359 effort=25 velocity=1.5 -> lower=-3.14159265359 upper=3.14159265359 effort=25 velocity=3.0
- joint lh_hip_joint: limit lower=-3.14159265359 upper=3.14159265359 effort=25 velocity=1.5 -> lower=-3.14159265359 upper=3.14159265359 effort=25 velocity=3.0
- joint lh_lower_leg_joint: limit lower=-3.14159265359 upper=3.14159265359 effort=25 velocity=1.5 -> lower=-3.14159265359 upper=3.14159265359 effort=25 velocity=3.0
- joint lh_upper_leg_joint: limit lower=-3.14159265359 upper=3.14159265359 effort=25 velocity=1.5 -> lower=-3.14159265359 upper=3.14159265359 effort=25 velocity=3.0
- joint rf_hip_joint: limit lower=-3.14159265359 upper=3.14159265359 effort=25 velocity=1.5 -> lower=-3.14159265359 upper=3.14159265359 effort=25 velocity=3.0
- joint rf_lower_leg_joint: limit lower=-3.14159265359 upper=3.14159265359 effort=25 velocity=1.5 -> lower=-3.14159265359 upper=3.14159265359 effort=25 velocity=3.0
- joint rf_upper_leg_joint: limit lower=-3.14159265359 upper=3.14159265359 effort=25 velocity=1.5 -> lower=-3.14159265359 upper=3.14159265359 effort=25 velocity=3.0
- joint rh_hip_joint: limit lower=-3.14159265359 upper=3.14159265359 effort=25 velocity=1.5 -> lower=-3.14159265359 upper=3.14159265359 effort=25 velocity=3.0
- joint rh_lower_leg_joint: limit lower=-3.14159265359 upper=3.14159265359 effort=25 velocity=1.5 -> lower=-3.14159265359 upper=3.14159265359 effort=25 velocity=3.0
- joint rh_upper_leg_joint: limit lower=-3.14159265359 upper=3.14159265359 effort=25 velocity=1.5 -> lower=-3.14159265359 upper=3.14159265359 effort=25 velocity=3.0

File: urdf/opendog.urdf.xacro (robot description, xacro)
@@ -15,5 +15,5 @@
             <origin xyz="0.25 0.185 0.002" rpy="0 0 1.5708" />
             <geometry>
-                <mesh filename="package://opendog_description/meshes/base.stl" scale="0.001 0.001 0.001" />
+                <mesh filename="${base_mesh_path}" scale="0.001 0.001 0.001" />
             </geometry>
             <material name="black" />
@@ -22,5 +22,5 @@
     <link name="base_inertia">
         <inertial>
-            <origin xyz="0 0 0" />
+            <origin xyz="-0.1 0 0" />
             <mass value="${base_mass}" />
             <inertia ixx="${(1/12) * base_mass * (base_y_length * base_y_length + base_z_length * base_z_length)}" ixy="0.0" ixz="0.0"
@@ -32,5 +32,5 @@
         <parent link="base_link"/>
         <child link="base_inertia"/>
-        <origin rpy="0 0 0" xyz="0 0 0"/>
+        <origin rpy="0 0 0" xyz="0.05 0 0"/>
     </joint>
     <gazebo reference="base_link">

File: urdf/properties.urdf.xacro (robot description, xacro)
@@ -16,16 +16,16 @@
     <xacro:property name="upper_leg_mesh_path" value="package://opendog_description/meshes/upper_leg.stl" />
     <xacro:property name="upper_leg_mass" value="0.125" />
-    <xacro:property name="upper_leg_x_length" value="0.05" />
-    <xacro:property name="upper_leg_y_length" value="0.03" />
-    <xacro:property name="upper_leg_z_length" value="0.1905" />
+    <xacro:property name="upper_leg_x_length" value="0.08" />
+    <xacro:property name="upper_leg_y_length" value="0.08" />
+    <xacro:property name="upper_leg_z_length" value="0.30" />
     <xacro:property name="lower_leg_mesh_path" value="package://opendog_description/meshes/lower_leg.stl" />
     <xacro:property name="lower_leg_mass" value="0.125" />
     <xacro:property name="lower_leg_x_length" value="0.039" />
     <xacro:property name="lower_leg_y_length" value="0.022" />
-    <xacro:property name="lower_leg_z_length" value="0.156" />
+    <xacro:property name="lower_leg_z_length" value="0.30" />
     <xacro:property name="base_mesh_path" value="package://opendog_description/meshes/base.stl" />
     <xacro:property name="base_mass" value="2.0" />
-    <xacro:property name="base_x_length" value="0.5" />
+    <xacro:property name="base_x_length" value="0.8" />
     <xacro:property name="base_y_length" value="0.29" />
-    <xacro:property name="base_z_length" value="0.130" />
+    <xacro:property name="base_z_length" value="0.22" />
 </robot>
